File: src/kicad/Light Sensor LED.kicad_pcb (KiCad board)
At the start: 2 copper layers, 88.2 x 72 mm, 15 parts, among them J1 USB_A, U1 NE555P

Commit message: Revised Project
Parts:
- C2: value 0.1u -> 0.01u
Other:
- board text added: "github.com/rocketblaster/Light-Sensor-LED"
- board text removed: "github.com/rocketblaster"
Changed lines of the file:
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@@
 			)
 		)
-		(property "Value" "0.1u"
+		(property "Value" "0.01u"
 			(at 2.5 3.75 0)
 			(layer "F.Fab")
@@
 		(layer "Edge.Cuts")
 	)
-	(gr_text "github.com/rocketblaster"
-		(at 159 117 0)
+	(gr_text "github.com/rocketblaster/Light-Sensor-LED"
+		(at 167 86 0)
 		(layer "B.SilkS")
 		(effects

Commit message: Revised Project
Parts:
- removed C3, C4: 10u, Capacitor_THT:C_Disc_D8.0mm_W5.0mm_P5.00mm
- moved R5 4.12 mm to (135.0, 106.0)
- moved U1 4.00 mm to (157.0, 111.0)
- moved R1 3.61 mm to (168.0, 97.0)
- moved C2 2.00 mm to (171.0, 105.0)
Connections:
- R5 pad 1: Net-(C3-Pad2) -> Net-(U1-OUT)
- R6 pad 1: Net-(C4-Pad2) -> Net-(U1-OUT)
Routing:
- net Net-(U1-OUT): track 31.3 -> 47.5 mm
- net Net-(C3-Pad2): track 7.57 -> 0.00 mm
- net Net-(C4-Pad2): track 6.62 -> 0.00 mm
- net Net-(U1-DISCH): track 17.0 -> 11.8 mm
- net Net-(U1-~{RST}): track 52.1 -> 56.9 mm
- net Net-(D1-A): track 12.2 -> 8.91 mm
- net Net-(U1-CONT): track 10.5 -> 7.64 mm
- net Net-(U1-THRES): track 37.1 -> 38.7 mm
- net VCC: track 58.2 -> 57.7 mm
